File: kicad-hardware/Sensor_Power_Baseboard/Sensor_Power_Baseboard/Sensor_Power_Baseboard.kicad_sch (KiCad schematic)
At the start: 0 parts

Commit message: feat(hardware): finalize PCB layout, add 3D renders, manufacturing Gerbers, and update portfolio
Parts:
- added C1: 10uF, Capacitor_SMD:C_0805_2012Metric, symbol Device:C
- added C2, C4: 100nF, Capacitor_SMD:C_0805_2012Metric, symbol Device:C
- added C3: 22uF, Capacitor_SMD:C_0805_2012Metric, symbol Device:C
- added D1: LED, LED_SMD:LED_0805_2012Metric, symbol Device:LED
- added J1: USB_C_Receptacle_USB2.0_16P, Connector_USB:USB_C_Receptacle_HRO_TYPE-C-31-M-12, symbol Connector:USB_C_Receptacle_USB2.0_16P
- added OledScreen1: Conn_01x04_Pin, Connector_PinHeader_2.54mm:PinHeader_1x04_P2.54mm_Vertical, symbol Connector:Conn_01x04_Pin
- added R1, R2: 5.1K, Resistor_SMD:R_0805_2012Metric, symbol Device:R
- added R3: 1k, Resistor_SMD:R_0805_2012Metric, symbol Device:R
- added R4, R5: 4.7k, Resistor_SMD:R_0805_2012Metric, symbol Device:R
- added U1: AMS1117-3.3, Package_TO_SOT_SMD:SOT-223-3_TabPin2, symbol Regulator_Linear:AMS1117-3.3
Connections:
- new net: J1.A5 (CC1), R1.1
- new net: J1.B5 (CC2), R2.1
- new net: D1.1 (K), R3.2
- new net: C3.2, D1.2 (A)
- new net +3V3: C3.1, C4.1, OledScreen1.1 (Pin_1), R4.1, R5.1, U1.2 (VO)
- new net +5V: C1.1, C2.2, J1.A4 (VBUS), J1.A9 (VBUS), J1.B4 (VBUS), J1.B9 (VBUS), U1.3 (VI)
- new net GND: C1.2, C2.1, C4.2, J1.A1 (GND), J1.A12 (GND), J1.B1 (GND), J1.B12 (GND), J1.SH (SHIELD), OledScreen1.2 (Pin_2), R1.2, R2.2, R3.1, U1.1 (GND)
- new net SCL: OledScreen1.4 (Pin_4), R5.2
- new net SDA: OledScreen1.3 (Pin_3), R4.2
- no-connect marks 0 -> 6
